Commit message: change camera angle

File: camera/kobuki.urdf.xacro (robot description, xacro)
@@ -235,5 +235,5 @@
   <joint name="custom_camera_joint_right" type="fixed">
     <axis xyz="0 1 0" />
-   <origin xyz=".12 .11 .153" rpy="0 0.4 0.4"/>
+   <origin xyz=".12 .11 .153" rpy="0 0.4 0.77"/>
     <parent link="base_link"/>
     <child link="left_camera"/>
@@ -263,5 +263,5 @@
   <joint name="custom_camera_joint_left" type="fixed">
     <axis xyz="0 1 0" />
-    <origin xyz=".12 -.11 .153" rpy="0 0.4 -0.4"/>
+    <origin xyz=".12 -.11 .153" rpy="0 0.4 -0.77"/>
     <parent link="base_link"/>
     <child link="right_camera"/>

Commit message: Z_course 3/4 chance it is possible

File: camera/kobuki.urdf.xacro (robot description, xacro)
@@ -235,5 +235,5 @@
   <joint name="custom_camera_joint_right" type="fixed">
     <axis xyz="0 1 0" />
-   <origin xyz=".12 .11 .153" rpy="0 0.4 0.77"/>
+   <origin xyz=".12 .11 .153" rpy="0 0.5 0.77"/>
     <parent link="base_link"/>
     <child link="left_camera"/>
@@ -263,5 +263,5 @@
   <joint name="custom_camera_joint_left" type="fixed">
     <axis xyz="0 1 0" />
-    <origin xyz=".12 -.11 .153" rpy="0 0.4 -0.77"/>
+    <origin xyz=".12 -.11 .153" rpy="0 0.5 -0.77"/>
     <parent link="base_link"/>
     <child link="right_camera"/>
